File: kicad/led_matrix_8x4_module.kicad_sch (KiCad schematic)
At the start: 64 parts, among them J1 Conn_01x04, J2 Conn_01x02_Female, J3 Conn_01x04_Female, J4 DIP_SOCKET_02x08, Q1 PN2222A, Q2 PN2222A, Q3 PN2222A, Q4 PN2222A, Q5 PN2222A, Q6 PN2222A, Q7 PN2222A, Q8 PN2222A, U1 74HC595

Commit message: release: v1.1
Parts:
- added C4: 0.1uf, Capacitor_THT:C_Disc_D3.0mm_W1.6mm_P2.50mm, symbol Device:C
- added H1, H2, H3, H4: MountingHole, MountingHole:MountingHole_2.2mm_M2_Pad_Via, symbol Mechanical:MountingHole
- C1: value 33uf -> 100uf; footprint Capacitor_THT:CP_Radial_D4.0mm_P2.00mm -> Capacitor_THT:CP_Radial_D5.0mm_P2.00mm
- C3: value 0.1uf -> 33uf
- D1, D10, D11, D12, D13, D14, D15, D16, D17, D18, D19, D2, D20, D21, D22, D23, D24, D25, D26, D27, D28, D29, D3, D30, D31, D32, D4, D5, D6, D7, D8, D9: footprint LED_THT:LED_Oval_W5.2mm_H3.8mm -> LED_THT:LED_D5.0mm
- J1, J3: footprint Connector_PinHeader_2.00mm:PinHeader_1x04_P2.00mm_Vertical -> Connector_PinHeader_2.00mm:PinHeader_1x04_P2.00mm_Horizontal
- J2: footprint Connector_PinHeader_2.00mm:PinHeader_1x02_P2.00mm_Vertical -> Connector_PinHeader_2.00mm:PinHeader_1x02_P2.00mm_Horizontal
- R1, R10, R11, R12, R13, R14, R15, R16, R2, R3, R4, R5, R6, R7, R8, R9: footprint Resistor_THT:R_Axial_DIN0204_L3.6mm_D1.6mm_P1.90mm_Vertical -> Resistor_THT:R_Axial_DIN0204_L3.6mm_D1.6mm_P5.08mm_Horizontal
Connections:
- net +5V: now also C4.1
- net GNDREF: now also C4.2
Other:
- note added: "Mounting Holes"
- moved on the sheet: C1, C2, C3, U1
